File: pcb/left/keyboard_pcb.kicad_sch (KiCad schematic)
At the start: 33 parts, among them J1 TRRS, K00 KEYSW, K01 KEYSW, K02 KEYSW, K03 KEYSW, K04 KEYSW, K05 KEYSW, K10 KEYSW, K11 KEYSW, K12 KEYSW, K13 KEYSW, K14 KEYSW, K15 KEYSW, K20 KEYSW, K21 KEYSW, K22 KEYSW, K23 KEYSW, K24 KEYSW, K25 KEYSW, K30 KEYSW, K31 KEYSW, K32 KEYSW, U2 Pico

Commit message: Switched to 0xCB Helios controller
Parts:
- removed MB1, MB2, MB3, MB4: MountingHole, beekeeb_lib:mousebites, symbol Mechanical:MountingHole
- removed R1: 5k6, Resistor_SMD:R_1206_3216Metric_Pad1.30x1.75mm_HandSolder, symbol Device:R
- removed R2: 10k, Resistor_SMD:R_1206_3216Metric_Pad1.30x1.75mm_HandSolder, symbol Device:R
- removed U2: Pico, RPi_Pico:RPi_Pico_SMD_TH, symbol KiCad-RP-Pico:Pico
- added U1: Helios, PCM_marbastlib-xp-promicroish:Helios_AH_USBdn, symbol PCM_marbastlib-promicroish:Helios
- J1: footprint Resistor_SMD:R_1206_3216Metric_Pad1.30x1.75mm_HandSolder -> Keebio-Parts:TRRS-PJ-320A
- K00, K01, K02, K03, K04, K05, K10, K11, K12, K13, K14, K15, K20, K21, K22, K23, K24, K25, K30, K31, K32: footprint keyswitches:SW_PG1350_reversible -> keyswitches:Kailh_socket_PG1350_optional
Connections:
- net GND: now also U1.14 (GND), U1.3 (GND), U1.4 (GND)
- net VCC: now also U1.13 (5V)
- net k00: now also U1.23 (P23)
- net k01: now also U1.22 (P20)
- net k02: now also U1.8 (P5)
- net k03: now also U1.7 (P4)
- net k04: now also U1.31 (P10)
- net k05: now also U1.30 (P11)
- net k10: now also U1.29 (P16)
- net k11: now also U1.24 (P21)
- net k12: now also U1.10 (P7)
- net k13: now also U1.9 (P6)
- net k14: now also U1.11 (P8)
- net k15: now also U1.17 (P29)
- net k20: now also U1.28 (P15)
- net k21: now also U1.27 (P14)
- net k22: now also U1.19 (P27)
- net k23: now also U1.18 (P28)
- net k24: now also U1.20 (P26)
- net k25: now also U1.21 (P22)
- net k30: now also U1.26 (P13)
- net k31: now also U1.25 (P12)
- net k32: now also U1.12 (P9)
- net rx: now also U1.2 (P1)
- net tx: now also U1.1 (P0)
- no-connect marks 9 -> 1
